Commit message: Rajagopal: Solved the navigation 2d pose estimation swawp

File: mybot_description/urdf/fork_redesigned_urdf.xacro (robot description, xacro)
@@ -65,5 +65,7 @@
   <joint name="base_joint" type="fixed">
     <parent link="base_footprint"/><child link="base_link"/>
-    <origin xyz="0 0 ${wheel_radius}" rpy="0 0 0"/>   <!-- base_link = wheel-axle midpoint -->
+    <!-- Yaw 180: the front panel is the front, the forks are the back.
+         Pose-estimate arrows follow +X, so +X must point at the front panel. -->
+    <origin xyz="0 0 ${wheel_radius}" rpy="0 0 ${pi}"/>
   </joint>
   <!-- Battery inside the lower chassis. CAD parts alone put the assembled
@@ -242,5 +244,6 @@
   <joint name="imu_joint" type="fixed">
     <parent link="imu_mount_link"/><child link="imu_link"/>
-    <origin xyz="0 0 0" rpy="0 0 ${pi/2}"/>
+    <!-- +X is the front panel, same as base_footprint, so IMU yaw matches the robot. -->
+    <origin xyz="0 0 0" rpy="0 0 ${-pi/2}"/>
   </joint>
   <!-- ===================== ROS2_CONTROL (same as mybot.urdf.xacro) ===================== -->
@@ -281,5 +284,5 @@
       <parameters>$(find mybot_gazebo)/config/fork_controllers.yaml</parameters>
       <ros>
-        <remapping>diff_drive_controller/odom:=/wheel_odom</remapping>
+        <remapping>diff_drive_controller/odom:=/odom</remapping>
         <remapping>diff_drive_controller/cmd_vel_unstamped:=/cmd_vel</remapping>
       </ros>
@@ -316,5 +319,6 @@
             <samples>180</samples>
             <resolution>1</resolution>
-            <!-- 90 deg to 270 deg. 0 is +X, toward the forks. -->
+            <!-- 90 deg to 270 deg in laser_link. That frame points at the
+                 forks (the back); this window faces the front panel. -->
             <min_angle>1.5708</min_angle>
             <max_angle>4.7124</max_angle>
