Commit message: Updated ROS2 packages

File: mybot_description/urdf/mybot.urdf.xacro (robot description, xacro)
@@ -1,14 +1,35 @@
 <?xml version="1.0"?>
 <robot name="mybot" xmlns:xacro="http://www.ros.org/wiki/xacro">
-  <xacro:property name="base_length" value="0.4"/>
-  <xacro:property name="base_width" value="0.3"/>
-  <xacro:property name="base_height" value="0.15"/>
-  <xacro:property name="wheel_radius" value="0.08"/>
-  <xacro:property name="wheel_width" value="0.04"/>
+  <!-- ============================================================
+       GEOMETRY — computed so body never touches ground.
+       Design rule:
+         wheel axle is at the BOTTOM FACE of base_link (z = -base_height/2
+         in base_link frame).  This guarantees body clears ground by
+         wheel_radius regardless of base_height.
+         base_joint lifts base_link so wheel bottoms touch ground:
+           base_joint_z = wheel_radius - wheel_offset_z
+                        = wheel_radius + base_height/2
+         Caster joint z is chosen so sphere bottom = wheel bottom.
+  ============================================================ -->
+  <xacro:property name="base_length"      value="0.4"/>
+  <xacro:property name="base_width"       value="0.3"/>
+  <xacro:property name="base_height"      value="0.15"/>
+  <xacro:property name="wheel_radius"     value="0.08"/>
+  <xacro:property name="wheel_width"      value="0.04"/>
   <xacro:property name="wheel_separation" value="0.34"/>
-  <xacro:property name="wheel_offset_x" value="0.0"/>
-  <xacro:property name="wheel_offset_z" value="-0.05"/>
-  <material name="grey"><color rgba="0.5 0.5 0.5 1"/></material>
-  <material name="black"><color rgba="0.1 0.1 0.1 1"/></material>
+  <!-- axle at base bottom face -->
+  <xacro:property name="wheel_offset_z"   value="${-base_height/2}"/>
+  <!-- caster: same radius as wheel so contact plane is identical -->
+  <xacro:property name="caster_radius"    value="0.05"/>
+  <!-- caster joint z so sphere bottom = ground:
+       base_link_z + caster_joint_z - caster_radius = 0 (ground at base_footprint z)
+       base_link_z = wheel_radius - wheel_offset_z = wheel_radius + base_height/2
+       caster_joint_z = caster_radius - base_link_z
+                      = caster_radius - wheel_radius - base_height/2             -->
+  <xacro:property name="caster_joint_z"  value="${caster_radius - wheel_radius - base_height/2}"/>
+  <!-- ============================================================ MATERIALS -->
+  <material name="grey"> <color rgba="0.5 0.5 0.5 1"/> </material>
+  <material name="black"><color rgba="0.1 0.1 0.1 1"/> </material>
+  <!-- ============================================================ BASE -->
   <link name="base_footprint"/>
   <link name="base_link">
@@ -22,12 +43,15 @@
     <inertial>
       <mass value="5.0"/>
-      <inertia ixx="0.06" ixy="0" ixz="0" iyy="0.08" iyz="0" izz="0.1"/>
+      <inertia ixx="0.0578" ixy="0" ixz="0"
+               iyy="0.0911" iyz="0"
+               izz="0.1156"/>
     </inertial>
   </link>
   <joint name="base_joint" type="fixed">
     <parent link="base_footprint"/>
-    <child link="base_link"/>
-    <origin xyz="0 0 ${wheel_radius}" rpy="0 0 0"/>
+    <child  link="base_link"/>
+    <origin xyz="0 0 ${wheel_radius - wheel_offset_z}" rpy="0 0 0"/>
   </joint>
+  <!-- ============================================================ WHEELS -->
   <xacro:macro name="wheel" params="prefix reflect">
     <link name="${prefix}_wheel_link">
@@ -43,39 +67,55 @@
       <inertial>
         <mass value="0.5"/>
-        <inertia ixx="0.001" ixy="0" ixz="0" iyy="0.001" iyz="0" izz="0.001"/>
+        <inertia ixx="0.00052" ixy="0" ixz="0"
+                 iyy="0.00063" iyz="0"
+                 izz="0.00052"/>
       </inertial>
     </link>
     <joint name="${prefix}_wheel_joint" type="continuous">
       <parent link="base_link"/>
-      <child link="${prefix}_wheel_link"/>
-      <origin xyz="${wheel_offset_x} ${reflect*wheel_separation/2} ${wheel_offset_z}" rpy="0 0 0"/>
+      <child  link="${prefix}_wheel_link"/>
+      <origin xyz="0 ${reflect * wheel_separation/2} ${wheel_offset_z}" rpy="0 0 0"/>
       <axis xyz="0 1 0"/>
+      <dynamics damping="0.2" friction="0.1"/>
+      <limit effort="10.0" velocity="10.0"/>
     </joint>
   </xacro:macro>
-  <xacro:wheel prefix="left" reflect="1"/>
+  <xacro:wheel prefix="left"  reflect="1"/>
   <xacro:wheel prefix="right" reflect="-1"/>
-  <link name="caster_wheel_link">
-    <visual>
-      <geometry><sphere radius="0.04"/></geometry>
-      <material name="black"/>
-    </visual>
-    <collision>
-      <geometry><sphere radius="0.04"/></geometry>
-    </collision>
-    <inertial>
-      <mass value="0.2"/>
-      <inertia ixx="0.0001" ixy="0" ixz="0" iyy="0.0001" iyz="0" izz="0.0001"/>
-    </inertial>
-  </link>
-  <joint name="caster_joint" type="fixed">
-    <parent link="base_link"/>
-    <child link="caster_wheel_link"/>
-    <origin xyz="${base_length/2 - 0.05} 0 -0.09" rpy="0 0 0"/>
-  </joint>
-  <!-- ============================================================ -->
-  <!-- ros2_control hardware interface                              -->
-  <!-- The controller_manager reads this block to know what joints -->
-  <!-- are available and what interfaces they expose.              -->
-  <!-- ============================================================ -->
+  <!-- ============================================================ CASTERS -->
+  <xacro:macro name="caster" params="prefix x_offset y_offset">
+    <link name="caster_${prefix}_link">
+      <visual>
+        <geometry><sphere radius="${caster_radius}"/></geometry>
+        <material name="black"/>
+      </visual>
+      <collision>
+        <geometry><sphere radius="${caster_radius}"/></geometry>
+      </collision>
+      <inertial>
+        <mass value="0.1"/>
+        <inertia ixx="0.0001" ixy="0" ixz="0"
+                 iyy="0.0001" iyz="0"
+                 izz="0.0001"/>
+      </inertial>
+    </link>
+    <joint name="caster_${prefix}_joint" type="fixed">
+      <parent link="base_link"/>
+      <child  link="caster_${prefix}_link"/>
+      <origin xyz="${x_offset} ${y_offset} ${caster_joint_z}" rpy="0 0 0"/>
+    </joint>
+    <gazebo reference="caster_${prefix}_link">
+      <material>Gazebo/Black</material>
+      <mu1>0.0</mu1>
+      <mu2>0.0</mu2>
+      <kp>100000.0</kp>
+      <kd>10.0</kd>
+      <minDepth>0.001</minDepth>
+      <maxVel>0.1</maxVel>
+    </gazebo>
+  </xacro:macro>
+  <xacro:caster prefix="front" x_offset="${ base_length/2 - 0.05}" y_offset="0.0"/>
+  <xacro:caster prefix="back"  x_offset="${-base_length/2 + 0.05}" y_offset="0.0"/>
+  <!-- ============================================================ ROS2_CONTROL -->
   <ros2_control name="GazeboSystem" type="system">
     <hardware>
@@ -99,51 +139,40 @@
     </joint>
   </ros2_control>
-  <!-- ============================================================ -->
-  <!-- Gazebo ros2_control plugin                                   -->
-  <!-- Bridges Gazebo joints into the ros2_control controller_manager -->
-  <!-- ============================================================ -->
+  <!-- ============================================================ GAZEBO PLUGINS -->
   <gazebo>
     <plugin name="gazebo_ros2_control" filename="libgazebo_ros2_control.so">
+      <robot_param>robot_description</robot_param>
+      <robot_param_node>robot_state_publisher</robot_param_node>
       <parameters>$(find mybot_gazebo)/config/controllers.yaml</parameters>
+      <ros>
+        <remapping>diff_drive_controller/odom:=/odom_raw</remapping>
+        <remapping>diff_drive_controller/cmd_vel_unstamped:=/cmd_vel</remapping>
+      </ros>
     </plugin>
-    <!-- Keep joint state publisher for wheel TF -->
-    <plugin name="joint_state_publisher" filename="libgazebo_ros_joint_state_publisher.so">
-      <ros><namespace>/</namespace></ros>
-      <update_rate>30</update_rate>
-      <joint_name>left_wheel_joint</joint_name>
-      <joint_name>right_wheel_joint</joint_name>
-    </plugin>
-  </gazebo>
-  <gazebo reference="base_link"><material>Gazebo/Grey</material></gazebo>
-  <gazebo reference="left_wheel_link"><material>Gazebo/Black</material></gazebo>
-  <gazebo reference="right_wheel_link"><material>Gazebo/Black</material></gazebo>
-  <xacro:macro name="caster" params="prefix x_offset">
-    <link name="caster_${prefix}_link">
-      <visual>
-        <geometry><sphere radius="0.04"/></geometry>
-        <material name="black"/>
-      </visual>
-      <collision>
-        <geometry><sphere radius="0.04"/></geometry>
-      </collision>
-      <inertial>
-        <mass value="0.2"/>
-        <inertia ixx="0.0001" ixy="0" ixz="0" iyy="0.0001" iyz="0" izz="0.0001"/>
-      </inertial>
-    </link>
-    <joint name="caster_${prefix}_joint" type="fixed">
-      <parent link="base_link"/>
-      <child link="caster_${prefix}_link"/>
-      <origin xyz="${x_offset} 0 -0.09" rpy="0 0 0"/>
-    </joint>
-    <gazebo reference="caster_${prefix}_link">
-      <material>Gazebo/Black</material>
-      <mu1>0.0</mu1>
-      <mu2>0.0</mu2>
-    </gazebo>
-  </xacro:macro>
-  <xacro:caster prefix="front" x_offset="${base_length/2 - 0.05}"/>
-  <xacro:caster prefix="back" x_offset="${-(base_length/2 - 0.05)}"/>
-<!-- ============ LIDAR ============ -->
+  </gazebo>
+  <!-- ============================================================ GAZEBO LINK PROPS -->
+  <gazebo reference="base_link">
+    <material>Gazebo/Grey</material>
+    <self_collide>false</self_collide>
+  </gazebo>
+  <gazebo reference="left_wheel_link">
+    <material>Gazebo/Black</material>
+    <mu1>1.0</mu1>
+    <mu2>1.0</mu2>
+    <kp>100000.0</kp>
+    <kd>10.0</kd>
+    <minDepth>0.001</minDepth>
+    <maxVel>0.1</maxVel>
+  </gazebo>
+  <gazebo reference="right_wheel_link">
+    <material>Gazebo/Black</material>
+    <mu1>1.0</mu1>
+    <mu2>1.0</mu2>
+    <kp>100000.0</kp>
+    <kd>10.0</kd>
+    <minDepth>0.001</minDepth>
+    <maxVel>0.1</maxVel>
+  </gazebo>
+  <!-- ============================================================ LIDAR -->
   <xacro:property name="lidar_radius" value="0.04"/>
   <xacro:property name="lidar_height" value="0.05"/>
@@ -158,11 +187,12 @@
     <inertial>
       <mass value="0.15"/>
-      <inertia ixx="0.0001" ixy="0" ixz="0" iyy="0.0001" iyz="0" izz="0.0001"/>
+      <inertia ixx="0.0001" ixy="0" ixz="0"
+               iyy="0.0001" iyz="0"
+               izz="0.0001"/>
     </inertial>
   </link>
   <joint name="laser_joint" type="fixed">
     <parent link="base_link"/>
-    <child link="laser_link"/>
-    <!-- centered on top of base_link -->
+    <child  link="laser_link"/>
     <origin xyz="0 0 ${base_height/2 + lidar_height/2}" rpy="0 0 0"/>
   </joint>
@@ -203,5 +233,5 @@
     </sensor>
   </gazebo>
-  <!-- ============ IMU ============ -->
+  <!-- ============================================================ IMU -->
   <xacro:property name="imu_size" value="0.02"/>
   <link name="imu_link">
@@ -210,17 +240,14 @@
       <material name="black"/>
     </visual>
-    <!-- no collision: IMU is a sensor mount, not a physical body.
-         Adding collision here overlaps base_link's own collision box
-         and causes ODE to violently resolve the interpenetration,
-         which is what produced the wheel vibration. -->
     <inertial>
       <mass value="0.001"/>
-      <inertia ixx="0.0000001" ixy="0" ixz="0" iyy="0.0000001" iyz="0" izz="0.0000001"/>
+      <inertia ixx="1e-7" ixy="0" ixz="0"
+               iyy="1e-7" iyz="0"
+               izz="1e-7"/>
     </inertial>
   </link>
   <joint name="imu_joint" type="fixed">
     <parent link="base_link"/>
-    <child link="imu_link"/>
-    <!-- mounted at the center of base_link -->
+    <child  link="imu_link"/>
     <origin xyz="0 0 0" rpy="0 0 0"/>
   </joint>
@@ -228,5 +255,4 @@
     <material>Gazebo/Black</material>
     <sensor name="imu_sensor" type="imu">
-      <pose>0 0 0 0 0 0</pose>
       <always_on>true</always_on>
       <update_rate>100</update_rate>

Commit message: Updated Slam mapping

File: mybot_description/urdf/mybot.urdf.xacro (robot description, xacro)
@@ -179,27 +179,28 @@
   <link name="laser_link">
     <visual>
-      <geometry><cylinder radius="${lidar_radius}" length="${lidar_height}"/></geometry>
+      <geometry>
+        <cylinder radius="${lidar_radius}" length="${lidar_height}"/>
+      </geometry>
       <material name="black"/>
     </visual>
-    <collision>
-      <geometry><cylinder radius="${lidar_radius}" length="${lidar_height}"/></geometry>
-    </collision>
     <inertial>
-      <mass value="0.15"/>
-      <inertia ixx="0.0001" ixy="0" ixz="0"
-               iyy="0.0001" iyz="0"
-               izz="0.0001"/>
+      <mass value="0.1"/>
+      <origin xyz="0 0 0"/>
+      <inertia
+        ixx="0.0001" ixy="0.0" ixz="0.0"
+        iyy="0.0001" iyz="0.0"
+        izz="0.0001"/>
     </inertial>
   </link>
   <joint name="laser_joint" type="fixed">
     <parent link="base_link"/>
-    <child  link="laser_link"/>
+    <child link="laser_link"/>
     <origin xyz="0 0 ${base_height/2 + lidar_height/2}" rpy="0 0 0"/>
   </joint>
   <gazebo reference="laser_link">
-    <material>Gazebo/Black</material>
+    <self_collide>false</self_collide>
     <sensor name="lidar_sensor" type="ray">
-      <pose>0 0 0 0 0 0</pose>
-      <visualize>false</visualize>
+      <always_on>true</always_on>
+      <visualize>true</visualize>
       <update_rate>30</update_rate>
       <ray>
@@ -215,5 +216,5 @@
           <min>0.12</min>
           <max>10.0</max>
-          <resolution>0.015</resolution>
+          <resolution>0.01</resolution>
         </range>
         <noise>
@@ -225,9 +226,18 @@
       <plugin name="laser_plugin" filename="libgazebo_ros_ray_sensor.so">
         <ros>
-          <namespace>/</namespace>
-          <remapping>~/out:=scan</remapping>
+          <remapping>~/out:=/scan</remapping>
         </ros>
+        <frame_name>laser_link</frame_name>
         <output_type>sensor_msgs/LaserScan</output_type>
-        <frame_name>laser_link</frame_name>
+        <!-- Ignore the robot's own links -->
+        <ignore>
+          <link>base_link</link>
+          <link>laser_link</link>
+          <link>left_wheel_link</link>
+          <link>right_wheel_link</link>
+          <link>caster_front_link</link>
+          <link>caster_back_left_link</link>
+          <link>caster_back_right_link</link>
+        </ignore>
       </plugin>
     </sensor>

Commit message: Raja:Removed the rtabmap package and modified the urdf

File: mybot_description/urdf/mybot.urdf.xacro (robot description, xacro)
@@ -1,8 +1,4 @@
 <?xml version="1.0"?>
 <robot name="mybot" xmlns:xacro="http://www.ros.org/wiki/xacro">
-  <!-- Camera is optional — only pulled in when use_camera:=true is passed
-       to xacro at robot_description-generation time (i.e. by rtabmap.launch.py) -->
-  <xacro:arg name="use_camera" default="false"/>
-  <xacro:include filename="$(find mybot_description)/urdf/camera.urdf.xacro"/>
   <!-- ============================================================
        GEOMETRY — computed so body never touches ground.
@@ -241,6 +237,5 @@
           <link>right_wheel_link</link>
           <link>caster_front_link</link>
-          <link>caster_back_left_link</link>
-          <link>caster_back_right_link</link>
+          <link>caster_back_link</link>
         </ignore>
       </plugin>
@@ -294,7 +289,3 @@
     </sensor>
   </gazebo>
-  <!-- ============================================================ CAMERA -->
-  <xacro:if value="$(arg use_camera)">
-    <xacro:depth_camera parent_link="base_link"/>
-  </xacro:if>
 </robot>

Commit message: Modified xacro and cmake path and modified params yaml for laser data

File: mybot_description/urdf/mybot.urdf.xacro (robot description, xacro)
@@ -230,13 +230,11 @@
         <frame_name>laser_link</frame_name>
         <output_type>sensor_msgs/LaserScan</output_type>
-        <!-- Ignore the robot's own links -->
-        <ignore>
-          <link>base_link</link>
-          <link>laser_link</link>
-          <link>left_wheel_link</link>
-          <link>right_wheel_link</link>
-          <link>caster_front_link</link>
-          <link>caster_back_link</link>
-        </ignore>
+        <!-- NOTE: libgazebo_ros_ray_sensor.so has no self-filtering option;
+             an <ignore> tag here would be silently ignored. Self-body
+             returns are removed downstream by scan_filter_node
+             (laser_filters/LaserScanBoxFilter) publishing /scan_filtered —
+             see mybot_slam/config/scan_filter.yaml. Always view/consume
+             /scan_filtered, not raw /scan, for anything downstream of
+             the robot's own footprint. -->
       </plugin>
     </sensor>

Commit message: Chnaged controller to mppi

File: mybot_description/urdf/mybot.urdf.xacro (robot description, xacro)
@@ -67,7 +67,7 @@
       <inertial>
         <mass value="0.5"/>
-        <inertia ixx="0.00052" ixy="0" ixz="0"
-                 iyy="0.00063" iyz="0"
-                 izz="0.00052"/>
+        <inertia ixx="0.000867" ixy="0" ixz="0"
+                 iyy="0.00016" iyz="0"
+                 izz="0.000867"/>
       </inertial>
     </link>
@@ -77,6 +77,6 @@
       <origin xyz="0 ${reflect * wheel_separation/2} ${wheel_offset_z}" rpy="0 0 0"/>
       <axis xyz="0 1 0"/>
-      <dynamics damping="0.2" friction="0.1"/>
-      <limit effort="10.0" velocity="10.0"/>
+      <dynamics damping="0.01" friction="0.0"/>
+      <limit effort="2.0" velocity="60.0"/>
     </joint>
   </xacro:macro>
@@ -160,5 +160,5 @@
     <mu1>1.0</mu1>
     <mu2>1.0</mu2>
-    <kp>100000.0</kp>
+    <kp>1000000.0</kp>
     <kd>10.0</kd>
     <minDepth>0.001</minDepth>
@@ -169,5 +169,5 @@
     <mu1>1.0</mu1>
     <mu2>1.0</mu2>
-    <kp>100000.0</kp>
+    <kp>1000000.0</kp>
     <kd>10.0</kd>
     <minDepth>0.001</minDepth>

Commit message: Added options in start.sh file

File: mybot_description/urdf/mybot.urdf.xacro (robot description, xacro)
@@ -78,5 +78,5 @@
       <axis xyz="0 1 0"/>
       <dynamics damping="0.01" friction="0.0"/>
-      <limit effort="2.0" velocity="60.0"/>
+      <limit effort="2.0" velocity="10.0"/>
     </joint>
   </xacro:macro>
